File: CPU_8080_IR82-VA86.kicad_pcb (KiCad board)
At the start: 2 copper layers, 85 x 65 mm, 58 parts, among them X1 Power, X2 Address, X3 Data, X4 Mode, X5 Control, X6 Clock, X7 M1

Commit message: Add files via upload
Parts:
- removed X7: M1, Connector_PinHeader_2.54mm:PinHeader_1x02_P2.54mm_Vertical
- R2, R7, R8, R9: value 10k -> 1k
- VD1: footprint Diode_SMD:D_SOD-123 -> Diode_SMD:D_SOD-323_HandSoldering
- moved C17 7.16 mm to (118.1, 123.5), turned to 0 degrees
- moved JP1 6.91 mm to (96.9, 117.1), turned to -90 degrees
- moved R10 5.64 mm to (90.1, 115.0)
Connections:
- net /READY renamed Net-(DD3-READY)
- net /Single_BCLK renamed /F2TTL
- net /Single_OSC_TTL renamed /OSC_TTL
- DD4 pad 16: /INTE -> unconnected-(DD4-INTE-Pad16)
- X5 pad 4: /INTE -> /~{WRQ}
Routing:
- net /INTE: track 45.2 -> 0.00 mm, vias 2 -> 0
- net /~{INTA}: track 28.0 -> 34.1 mm
- net +12: track 116.2 -> 110.6 mm
- net /D5: track 40.1 -> 37.2 mm
- net Net-(JP1-A): track 4.58 -> 6.74 mm
- net /HLDA: track 88.0 -> 86.7 mm
- net /~{RESIN}: track 47.2 -> 46.3 mm
- net GND: vias 605 -> 632
Other:
- board text added: "v.1.3 24/03/2026"
- board text added: "~{WRQ}"
- board text removed: "Addr."
- board text removed: "INTE"
- board text removed: "v.1.2 21/12/2025"
