File: CPU_8080_IR82-VA86.kicad_sch (KiCad schematic)
At the start: 55 parts, among them X1 Power, X2 Address, X3 Data, X4 Mode, X5 Control, X6 Clock, X7 M1

Commit message: Add files via upload
Parts:
- removed X7: M1, Connector_PinHeader_2.54mm:PinHeader_1x02_P2.54mm_Vertical, symbol Connector_Generic:Conn_01x02
- R2, R7, R8, R9: value 10k -> 1k
- VD1: footprint Diode_SMD:D_SOD-123 -> Diode_SMD:D_SOD-323_HandSoldering
Connections:
- net INTE: no longer names the net of DD4.16 (INTE)
- net INTE: no longer X5.4 (Pin_4)
- net READY: no longer names the net of DD3.4 (READY), DD4.23 (READY)
- net Single_BCLK renamed F2TTL
- net Single_OSC_TTL renamed OSC_TTL
- new net ~{WRQ}: X5.4 (Pin_4)
- no-connect marks 5 -> 6
Other:
- note added: "Optional protector"
- note removed: "Future option"
- title: Модуль процессорный 580ВМ80 -> Модуль процессорный\n 580ВМ80
- moved on the sheet: C10, C3, C6, C7, C8, C9, DD3, R2, R3, R4, R5, SB1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
